File: Neve NKK JB switches.kicad_pcb (KiCad board)
At the start: 2 copper layers, 29.9 x 52.3 mm, 9 parts

Commit message: small updates
Other:
- board text added: "ess-103-x-03 03 on the end is a 8.38mm stand-off"
- board text added: "https://www.mouser.co.uk/datasheet/3/85/1/ess.pdf"
Changed lines of the file:
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@@
 		)
 	)
-	(gr_text "Button\nto base of \ncap"
-		(at 179.176573 114.879585 90)
+	(gr_text "ess-103-x-03\n03 on the end is a 8.38mm stand-off"
+		(at 241 108 0)
 		(layer "Dwgs.User")
 		(effects
@@
 		)
 	)
+	(gr_text "https://www.mouser.co.uk/datasheet/3/85/1/ess.pdf"
+		(at 208 104 0)
+		(layer "Dwgs.User")
+		(effects
+			(font
+				(size 1 1)
+				(thickness 0.15)
+			)
+			(justify left bottom)
+		)
+	)
+	(gr_text "Button\nto base of \ncap"
+		(at 179.176573 114.879585 90)
+		(layer "Dwgs.User")
+		(effects
+			(font
+				(size 1 1)
+				(thickness 0.15)
+			)
+			(justify left bottom)
+		)
+	)
 	(dimension
 		(type orthogonal)
@@
 		(layer "Dwgs.User")
 		(pts
+			(xy 107.877082 120) (xy 123 120.8551)
+		)
+		(height 24)
+		(orientation 0)
+		(format
+			(prefix "")
+			(suffix "")
+			(units 3)
+			(units_format 0)
+			(precision 4)
+			(suppress_zeroes yes)
+		)
+		(style
+			(thickness 0.1)
+			(arrow_length 1.27)
+			(text_position_mode 0)
+			(arrow_direction outward)
+			(extension_height 0.58642)
+			(extension_offset 0.5)
+			(keep_text_aligned yes)
+		)
+		(gr_text "15.1229"
+			(at 115.438541 142.85 0)
+			(layer "Dwgs.User")
+			(effects
+				(font
+					(size 1 1)
+					(thickness 0.15)
+				)
+			)
+		)
+	)
+	(dimension
+		(type orthogonal)
+		(layer "Dwgs.User")
+		(pts
 			(xy 174.176573 106.479585) (xy 174.176573 121.179585)
 		)
@@
 		(layer "Dwgs.User")
 		(pts
+			(xy 120.523 91.948) (xy 119.4 71.882)
+		)
+		(height 14.732)
+		(orientation 1)
+		(format
+			(prefix "")
+			(suffix "")
+			(units 3)
+			(units_format 0)
+			(precision 4)
+			(suppress_zeroes yes)
+		)
+		(style
+			(thickness 0.05)
+			(arrow_length 1.27)
+			(text_position_mode 0)
+			(arrow_direction outward)
+			(extension_height 0.58642)
+			(extension_offset 0.5)
+			(keep_text_aligned yes)
+		)
+		(gr_text "20.066"
+			(at 134.105 81.915 90)
+			(layer "Dwgs.User")
+			(effects
+				(font
+					(size 1 1)
+					(thickness 0.15)
+				)
+			)
+		)
+	)
+	(dimension
+		(type orthogonal)
+		(layer "Dwgs.User")
+		(pts
 			(xy 179.176573 106.479585) (xy 183.623999 97.811146)
 		)
@@
 		(layer "Dwgs.User")
 		(pts
-			(xy 123 121.92) (xy 92.964 121.92)
+			(xy 123 121.92) (xy 93.139902 120.839897)
 		)
 		(height 7.08)
@@
 			(keep_text_aligned yes)
 		)
-		(gr_text "30.036"
-			(at 107.982 127.85 0)
+		(gr_text "29.8601"
+			(at 108.069951 127.85 0)
 			(layer "Dwgs.User")
 			(effects
@@
 		(layer "Dwgs.User")
 		(pts
+			(xy 93.139902 120.870303) (xy 107.877082 121.13)
+		)
+		(height 23.129697)
+		(orientation 0)
+		(format
+			(prefix "")
+			(suffix "")
+			(units 3)
+			(units_format 0)
+			(precision 4)
+			(suppress_zeroes yes)
+		)
+		(style
+			(thickness 0.1)
+			(arrow_length 1.27)
+			(text_position_mode 0)
+			(arrow_direction outward)
+			(extension_height 0.58642)
+			(extension_offset 0.5)
+			(keep_text_aligned yes)
+		)
+		(gr_text "14.7372"
+			(at 100.508492 142.85 0)
+			(layer "Dwgs.User")
+			(effects
+				(font
+					(size 1 1)
+					(thickness 0.15)
+				)
+			)
+		)
+	)
+	(dimension
+		(type orthogonal)
+		(layer "Dwgs.User")
+		(pts
+			(xy 107.877082 120) (xy 118.03019 120.583682)
+		)
+		(height -3)
+		(orientation 0)
+		(format
+			(prefix "")
+			(suffix "")
+			(units 3)
+			(units_format 0)
+			(precision 4)
+			(suppress_zeroes yes)
+		)
+		(style
+			(thickness 0.1)
+			(arrow_length 1.27)
+			(text_position_mode 0)
+			(arrow_direction outward)
+			(extension_height 0.58642)
+			(extension_offset 0.5)
+			(keep_text_aligned yes)
+		)
+		(gr_text "10.1531"
+			(at 112.953636 115.85 0)
+			(layer "Dwgs.User")
+			(effects
+				(font
+					(size 1 1)
+					(thickness 0.15)
+				)
+			)
+		)
+	)
+	(dimension
+		(type orthogonal)
+		(layer "Dwgs.User")
+		(pts
+			(xy 107.877082 120.63) (xy 97.4598 121)
+		)
+		(height -3.63)
+		(orientation 0)
+		(format
+			(prefix "")
+			(suffix "")
+			(units 3)
+			(units_format 0)
+			(precision 4)
+			(suppress_zeroes yes)
+		)
+		(style
+			(thickness 0.1)
+			(arrow_length 1.27)
+			(text_position_mode 0)
+			(arrow_direction outward)
+			(extension_height 0.58642)
+			(extension_offset 0.5)
+			(keep_text_aligned yes)
+		)
+		(gr_text "10.4173"
+			(at 102.668441 115.85 0)
+			(layer "Dwgs.User")
+			(effects
+				(font
+					(size 1 1)
+					(thickness 0.15)
+				)
+			)
+		)
+	)
+	(dimension
+		(type orthogonal)
+		(layer "Dwgs.User")
+		(pts
 			(xy 97.4598 120.5738) (xy 99.9998 120.5992)
 		)
@@
 			(effects
 				(font
-					(size 1 1)
-					(thickness 0.15)
-				)
-			)
-		)
-	)
-	(dimension
-		(type orthogonal)
-		(layer "Edge.Cuts")
-		(pts
-			(xy 120.523 91.948) (xy 119.4 71.882)
-		)
-		(height 14.732)
-		(orientation 1)
-		(format
-			(prefix "")
-			(suffix "")
-			(units 3)
-			(units_format 0)
-			(precision 4)
-			(suppress_zeroes yes)
-		)
-		(style
-			(thickness 0.05)
-			(arrow_length 1.27)
-			(text_position_mode 0)
-			(arrow_direction outward)
-			(extension_height 0.58642)
-			(extension_offset 0.5)
-			(keep_text_aligned yes)
-		)
-		(gr_text "20.066"
-			(at 134.105 81.915 90)
-			(layer "Edge.Cuts")
-			(effects
-				(font
